Commit message: updates

File: src/my_robot_description/urdf/arm.xacro (robot description, xacro)
@@ -8,5 +8,4 @@
     <xacro:property name="hand_radius" value="0.02" />
     <xacro:property name="hand_length" value="0.3" />
-    <xacro:property name="base_height" value="0.02" />
     <link name="arm_base_link">
         <visual>
@@ -15,5 +14,5 @@
             </geometry>
             <origin xyz="0 0 ${arm_base_height / 2.0}" rpy="0 0 0" />
-            <material name="orange"/>
+            <material name="orange" />
         </visual>
         <collision>
@@ -21,12 +20,13 @@
                 <box size="${arm_base_length} ${arm_base_width} ${arm_base_height}" />
             </geometry>
+            <origin xyz="0 0 ${arm_base_height / 2.0}" rpy="0 0 0" />
         </collision>
         <xacro:box_inertia m="0.5" x="${arm_base_length}" y="${arm_base_width}" z="${arm_base_height}"
                            o_xyz="0 0 ${arm_base_height / 2.0}" o_rpy="0 0 0" />
     </link>
-      <link name="forearm_link">
+    <link name="forearm_link">
         <visual>
             <geometry>
-                <cylinder radius="${forearm_radius}" length="${forearm_length}"  />
+                <cylinder radius="${forearm_radius}" length="${forearm_length}" />
             </geometry>
             <origin xyz="0 0 ${forearm_length / 2.0}" rpy="0 0 0" />
@@ -37,15 +37,16 @@
                 <cylinder radius="${forearm_radius}" length="${forearm_length}" />
             </geometry>
+            <origin xyz="0 0 ${forearm_length / 2.0}" rpy="0 0 0" />
         </collision>
-        <xacro:cylinder_inertia  m="0.3" r="${forearm_radius}" l="${forearm_length}"
-                           o_xyz="0 0 ${forearm_length / 2.0}" o_rpy="0 0 0" />
+        <xacro:cylinder_inertia m="0.3" r="${forearm_radius}" l="${forearm_length}"
+                                o_xyz="0 0 ${forearm_length / 2.0}" o_rpy="0 0 0" />
     </link>
-      <link name="hand_link">
+    <link name="hand_link">
         <visual>
             <geometry>
-                <cylinder radius="${hand_radius}" length="${hand_length}"  />
+                <cylinder radius="${hand_radius}" length="${hand_length}" />
             </geometry>
             <origin xyz="0 0 ${hand_length / 2.0}" rpy="0 0 0" />
-            <material name="yellow" />
+            <material name="orange" />
         </visual>
         <collision>
@@ -53,28 +54,24 @@
                 <cylinder radius="${hand_radius}" length="${hand_length}" />
             </geometry>
+            <origin xyz="0 0 ${hand_length / 2.0}" rpy="0 0 0" />
         </collision>
-        <xacro:cylinder_inertia  m="0.3" r="${hand_radius}" l="${hand_length}"
-                           o_xyz="0 0 0" o_rpy="0 0 0" />
+        <xacro:cylinder_inertia m="0.3" r="${hand_radius}" l="${hand_length}"
+                                o_xyz="0 0 ${hand_length / 2.0}" o_rpy="0 0 0" />
     </link>
-    <!-- <joint name="base_arm_base_joint" type="fixed">
-        <parent link="base_link" />
-        <child link="arm_base_link" />
-        <origin xyz="${(base_length)/2.5} 0 ${base_height}" rpy="0 0 0" />
-    </joint> -->
-      <joint name="forearm_joint" type="revolute">
+    <joint name="arm_base_forearm_joint" type="revolute">
         <parent link="arm_base_link" />
         <child link="forearm_link" />
         <origin xyz="0 0 ${arm_base_height}" rpy="0 0 0" />
-        <axis xyz="0 1 0"/>
-        <limit lower="0" upper="${pi/2}" effort="100" velocity="100"/>
-        <dynamics friction="0.3" damping="0.3"/>
-     </joint>
-    <joint name="hand_joint" type="revolute">
-      <parent link="forearm_link" />
-      <child link="hand_link" />
-      <origin xyz="0 0 ${forearm_length}" rpy="0 0 0" />
-      <axis xyz="0 1 0"/>
-      <limit lower="0" upper="${pi/2}" effort="100" velocity="100"/>
-      <dynamics friction="0.3" damping="0.3"/>
+        <axis xyz="0 1 0" />
+        <limit lower="0" upper="${pi/2}" effort="100" velocity="100" />
+        <dynamics friction="0.3" damping="0.3" />
+    </joint>
+    <joint name="forearm_hand_joint" type="revolute">
+        <parent link="forearm_link" />
+        <child link="hand_link" />
+        <origin xyz="0 0 ${forearm_length}" rpy="0 0 0" />
+        <axis xyz="0 1 0" />
+        <limit lower="0" upper="${pi/2}" effort="100" velocity="100" />
+        <dynamics friction="0.3" damping="0.3" />
     </joint>
 </robot>

File: src/my_robot_description/urdf/common_properties.xacro (robot description, xacro)
@@ -7,9 +7,9 @@
         <color rgba="0.5 0.5 0.5 1" />
     </material>
-    <material name= "orange">
-         <color rgba="1 0.5 0 1" />
+    <material name="orange">
+        <color rgba="1.0 0.5 0 1" />
     </material>
-        <material name= "yellow">
-         <color rgba="1 0.75 0 1" />
+    <material name="yellow">
+        <color rgba="1.0 1.0 0 1" />
     </material>
     <xacro:macro name="box_inertia" params="m x y z o_xyz o_rpy">

File: src/my_robot_description/urdf/mobile_base.xacro (robot description, xacro)
@@ -13,5 +13,5 @@
             </geometry>
             <origin xyz="0 0 ${base_height / 2.0}" rpy="0 0 0" />
-            <material name="grey" />
+            <material name="blue" />
         </visual>
         <collision>
@@ -31,5 +31,5 @@
                 </geometry>
                 <origin xyz="0 0 0" rpy="${pi / 2.0} 0 0" />
-                <material name="red" />
+                <material name="grey" />
             </visual>
             <collision>

File: src/my_robot_description/urdf/my_robot.urdf.xacro (robot description, xacro)
@@ -5,4 +5,3 @@
     <xacro:include filename="mobile_base_gazebo.xacro" />
     <xacro:include filename="camera.xacro" />
-    <!-- <xacro:include filename="arm.xacro" /> -->
 </robot>

File: src/my_robot_description/urdf/standalone_arm.urdf.xacro (robot description, xacro)
@@ -1,5 +1,5 @@
 <?xml version="1.0"?>
 <robot name="my_robot" xmlns:xacro="http://www.ros.org/wiki/xacro">
-    <xacro:include filename="common_properties.xacro"/>
-    <xacro:include filename="arm.xacro"/>
+    <xacro:include filename="common_properties.xacro" />
+    <xacro:include filename="arm.xacro" />
 </robot>
